Commit message: Added python scripts to run package

File: urdf/humanSubject06_48dof.urdf (robot description, URDF)
Before this commit: robot XSensStyleModel_template, 49 links, 46 joints
Joints:
- added joint leftInnerShoulder_rotx: type revolute, parent T8, child LeftShoulder, origin xyz=0    0.029713    0.065446 rpy=0 0 0, axis 1 0 0, limit lower=-0.0872665 upper=0.785398 effort=30 velocity=1.0
- added joint rightShoulder_rotx: type revolute, parent RightShoulder, child RightUpperArm_f1, origin xyz=0    -0.15771           0 rpy=0 0 0, axis 1 0 0, limit lower=-2.35619 upper=1.5708 effort=30 velocity=1.0
- joint rightInnerShoulder_rotx: child RightUpperArm_f1 -> RightShoulder; limit lower=-2.35619 upper=1.5708 effort=30 velocity=1.0 -> lower=-0.785398 upper=0.0872665 effort=30 velocity=1.0; origin xyz=0    -0.15771           0 rpy=0 0 0 -> xyz=0   -0.029713    0.065446 rpy=0 0 0; parent RightShoulder -> T8
